Commit message: Added simplified Apto robot

File: urdf/robot.urdf (robot description, URDF)
Before this commit: robot apto_urdf, 26 links, 25 joints
Links:
- added link camera, mass 1e-9
- added link tcp_left, mass 1e-9
- added link tcp_right, mass 1e-9
Joints:
- added joint camera_frame: type fixed, parent servo_frame_3, child camera, origin xyz=-0.01795 0.0499 0.0361 rpy=-0 -1.5708 0, axis 0 0 0
- added joint tcp_left_frame: type fixed, parent gripper_frame, child tcp_left, origin xyz=-0.130554 0 0.01875 rpy=3.14159 1.5708 0, axis 0 0 0
- added joint tcp_right_frame: type fixed, parent gripper_frame_2, child tcp_right, origin xyz=-0.130554 0 -0.01875 rpy=3.14159 1.5708 0, axis 0 0 0
- joint gripper_carrier_left_1_frame: origin xyz=-0.0648039 -0.00825 -0.01125 rpy=3.14159 0 0 -> xyz=-0.0648039 0.00825 0.02905 rpy=-0 -0 0
- joint gripper_carrier_left_2_frame: origin xyz=-0.0648039 0.00825 0.04875 rpy=-0 0 0 -> xyz=-0.0648039 -0.00825 0.00845 rpy=3.14159 -0 0
- joint gripper_carrier_right_1_frame: origin xyz=-0.0648039 -0.00825 -0.01125 rpy=3.14159 -0 -0 -> xyz=-0.0648039 0.00825 -0.00845 rpy=0 0 -0
- joint gripper_carrier_right_2_frame: origin xyz=-0.0648039 0.00825 0.04875 rpy=0 -0 -0 -> xyz=-0.0648039 -0.00825 -0.02905 rpy=-3.14159 0 -0
- joint gripper_key_left_1: limit lower=-0.0197 upper=0 effort=10 velocity=10 -> lower=-0 upper=0.0197 effort=10 velocity=10; mimic (none) -> joint=gripper_key_left_2 multiplier=1.0; origin xyz=-0.0648039 0.00825 0.04875 rpy=-0 0 -0 -> xyz=-0.0648039 -0.00825 0.00845 rpy=3.14159 -0 0
- joint gripper_key_left_1_frame: origin xyz=0 0 0 rpy=0 0 0 -> xyz=0 0 -0 rpy=-0 0 -0
- joint gripper_key_left_2: limit lower=-0.0197 upper=-0 effort=10 velocity=10 -> lower=0 upper=0.0197 effort=10 velocity=10; mimic joint=gripper_key_left_1 multiplier=1.0 -> (none); origin xyz=-0.0648039 -0.00825 -0.01125 rpy=3.14159 0 0 -> xyz=-0.0648039 0.00825 0.02905 rpy=-0 -0 0
- joint gripper_key_left_2_frame: origin xyz=0 -0 0 rpy=0 0 -0 -> xyz=-0 0 0 rpy=-0 -0 0
- joint gripper_key_right_1: limit lower=-0.0197 upper=-0 effort=10 velocity=10 -> lower=-0 upper=0.0197 effort=10 velocity=10; mimic (none) -> joint=gripper_key_right_2 multiplier=1.0; origin xyz=-0.0648039 -0.00825 -0.01125 rpy=3.14159 -0 -0 -> xyz=-0.0648039 0.00825 -0.00845 rpy=0 0 0
- joint gripper_key_right_1_frame: origin xyz=0 -0 0 rpy=0 -0 0 -> xyz=0 0 0 rpy=0 0 0
- joint gripper_key_right_2: limit lower=-0.0197 upper=-0 effort=10 velocity=10 -> lower=-0 upper=0.0197 effort=10 velocity=10; mimic joint=gripper_key_right_1 multiplier=1.0 -> (none); origin xyz=-0.0648039 0.00825 0.04875 rpy=-0 -0 -0 -> xyz=-0.0648039 -0.00825 -0.02905 rpy=-3.14159 0 0
- joint gripper_key_right_2_frame: origin xyz=0 0 0 rpy=0 -0 0 -> xyz=0 0 0 rpy=0 0 0
- joint left_1: origin xyz=0.06435 0 0.238625 rpy=-1.1e-11 -1.5708 0 -> xyz=0.06435 0 0.238625 rpy=-1.5708 0 1.5708
- joint left_2: origin xyz=-0.0185 -0.0183 -0.03255 rpy=-1.5708 -0 3.14159 -> xyz=-0.0183 0.0185 -0.03255 rpy=-1.5708 0 1.5708
- joint left_3: origin xyz=0.09766 0 -0.018425 rpy=1.5708 -1.1e-11 -1.5708 -> xyz=0.09766 0 -0.018425 rpy=1.5708 -0 -1.5708
- joint left_4: origin xyz=-0.01915 0.01995 -0.0195 rpy=-1.5708 0 -1.5708 -> xyz=-0.01915 0.01995 -0.0195 rpy=-1.5708 -0 -1.5708
- joint left_5: origin xyz=-0.0566039 -0 0.01875 rpy=0 1.5708 0 -> xyz=-0.0566039 -0 0.01875 rpy=-0 1.5708 0
- joint left_6: origin xyz=-0.01825 0 -0.0422 rpy=-3.14159 -1.5708 0 -> xyz=0.01925 0 -0.0422 rpy=0 -1.5708 0
- joint right_1: origin xyz=-0.06435 2e-12 0.238625 rpy=-1.5708 0 -1.5708 -> xyz=-0.06435 2e-12 0.238625 rpy=1.5708 -0 -1.5708
- joint right_2: limit lower=-1.5708 upper=0.261799 effort=10 velocity=10 -> lower=-0.261799 upper=1.5708 effort=10 velocity=10; origin xyz=0.0183 0.0185 -0.03255 rpy=1.5708 -0 1.5708 -> xyz=0.0183 -0.0185 0.03255 rpy=1.5708 0 -1.5708
- joint right_3: origin xyz=0.09766 0 -0.019175 rpy=-1.5708 0 1.5708 -> xyz=0.09766 0 0.019175 rpy=-1.5708 0 -1.5708
- joint right_4: limit lower=-1.0472 upper=1.5708 effort=10 velocity=10 -> lower=-1.5708 upper=1.0472 effort=10 velocity=10; origin xyz=-0.0186 -0.0211 -0.0195 rpy=1.5708 -0 1.5708 -> xyz=-0.01905 0.0211 0.0195 rpy=1.5708 0 -1.5708
- joint right_5: origin xyz=-0.0558539 0 0.01875 rpy=0 1.5708 0 -> xyz=-0.0566039 -0 -0.01875 rpy=-0 -1.5708 0
- joint right_6: origin xyz=0.01915 -0 -0.0422 rpy=0 -1.5708 0 -> xyz=0.01915 -0 0.0422 rpy=0 1.5708 0
